Commit message: Using STOMP with ur5_2_moveit_config and ros kinetic

File: otim_traj/urdf/plugin.gazebo.xacro (robot description, xacro)
@@ -3,6 +3,7 @@
   <gazebo>
     <plugin name="ros_control" filename="libgazebo_ros_control.so">
-      <!-- <robotNamespace></robotNamespace>
-      <robotSimType>cob_gazebo_ros_control/HWISwitchRobotHWSim</robotSimType> -->
+      <!-- <robotNamespace></robotNamespace> -->
+      <robotSimType>gazebo_ros_control/DefaultRobotHWSim</robotSimType>
+      <legacyModeNS>true</legacyModeNS>
     </plugin>
   </gazebo>

File: otim_traj/urdf/ur5_grasp.urdf.xacro (robot description, xacro)
@@ -22,10 +22,10 @@
   <!-- Frame coincident with all-zeros TCP on UR controller -->
   <xacro:property name="tool0_offset" value="0.15"/>
-  <!-- <link name="grasping_link"/>
+  <link name="grasping_link"/>
   <joint name="ur5_joint_grasping_frame" type="fixed">
     <origin xyz="0 0 ${tool0_offset}" rpy="0 0 0"/>
     <parent link="tool0"/>
     <child link="grasping_link"/>
-  </joint> -->
+  </joint>
   ########################################
   # CAN Support code
