Commit message: add moveit_config to arm and endeffector

File: otim_traj/urdf/ur5_grasp.urdf.xacro (robot description, xacro)
@@ -20,17 +20,10 @@
   <!-- Frame coincident with all-zeros TCP on UR controller -->
   <xacro:property name="tool0_offset" value="0.15"/>
-  <link name="grasping_link"/>
+  <!-- <link name="grasping_link"/>
   <joint name="ur5_joint_grasping_frame" type="fixed">
     <origin xyz="0 0 ${tool0_offset}" rpy="0 0 0"/>
     <parent link="tool0"/>
     <child link="grasping_link"/>
-  </joint>
-  <!-- This frame is placed in the same position as the box inserted in Gazebo in order to be visualized in RVIZ (just for comparison) -->
-  <link name="reference_link"/>
-  <joint name="reference_frame" type="fixed">
-    <origin xyz="-0.5 0.1 0.05" rpy="0 0 -0.6"/>
-    <parent link="base_link"/>
-    <child link="reference_link"/>
-  </joint>
+  </joint> -->
   ########################################
   # Robotiq code

Commit message: Using camera to detect obstacles

File: otim_traj/urdf/ur5_grasp.urdf.xacro (robot description, xacro)
@@ -10,4 +10,6 @@
   <!-- It is necessary to change the hardware interface on the fly -->
   <!-- <xacro:include filename="$(find otim_traj)/urdf/ur5.transmission.xacro"/> -->
+  <!-- camera -->
+   <xacro:include filename="$(find otim_traj)/urdf/_d435.urdf.xacro" />
   <!-- arm -->
   <xacro:ur5_robot prefix="" joint_limited="false" transmission_hw_interface="$(arg transmission_hw_interface)"/>
@@ -26,4 +28,39 @@
     <child link="grasping_link"/>
   </joint> -->
+  ########################################
+  # CAN Support code
+  ########################################
+  <!-- o wrist 2 fica 0.09465 m abaixo de wrist 3 (-0.0445+0.09465)-->
+  <!-- Its position is relative to its own (Caution: treat as inverse direction)-->
+  <!-- Its orientation is relative to the previous frame -->
+  <link name="CAM_support_link">
+    <visual>
+      <!-- The cam is rotated 14 degrees (0.24rad) through the yaw axis -->
+      <origin rpy="${1.57 - 0.244} ${3.14} -1.57" xyz="${0.002 - 0.03} ${-0.023 + 0.03 - 0.01} ${0.13915-0.205}"/>
+      <geometry>
+        <mesh filename="package://otim_traj/model/cam_support/CAM_support.STL" scale="0.001 0.001 0.001"/>
+      </geometry>
+      <material name="Cyan">
+        <color rgba="0.91 0.91 0.88 1.0"/>
+      </material>
+    </visual>
+  </link>
+  <joint name="CAM_support_joint" type="fixed">
+    <origin rpy="0 ${0.244} 1.57" xyz="${-0.021 + 0.03 - 0.01} ${-0.027 + 0.03 + 0.015} ${0.205 - 0.0086}"/>
+    <parent link="wrist_2_link"/>
+    <child link="CAM_support_link"/>
+  </joint>
+  ########################################
+  # Realsense code
+  ########################################
+  <sensor_d435 parent="CAM_support_link">
+    <origin xyz="-0.0277 -0.002 -0.0075" rpy="0 0 0"/>
+  </sensor_d435>
+  <link name="d435_realsense"/>
+  <joint name="wrist3_camera" type="fixed">
+    <parent link="wrist_3_link"/>
+    <child link="d435_realsense"/>
+    <origin xyz="0.0 0.0 0.0" rpy="0.0 0.0 0.0"/>
+  </joint>
   ########################################
   # Robotiq code

Commit message: usando modelo de obstaculos no rviz

File: otim_traj/urdf/ur5_grasp.urdf.xacro (robot description, xacro)
@@ -34,8 +34,8 @@
   <!-- Its position is relative to its own (Caution: treat as inverse direction)-->
   <!-- Its orientation is relative to the previous frame -->
-  <link name="CAM_support_link">
-    <visual>
+  <!-- <link name="CAM_support_link">
+    <visual> -->
       <!-- The cam is rotated 14 degrees (0.24rad) through the yaw axis -->
-      <origin rpy="${1.57 - 0.244} ${3.14} -1.57" xyz="${0.002 - 0.03} ${-0.023 + 0.03 - 0.01} ${0.13915-0.205}"/>
+      <!-- <origin rpy="${1.57 - 0.244} ${3.14} -1.57" xyz="${0.002 - 0.03} ${-0.023 + 0.03 - 0.01} ${0.13915-0.205}"/>
       <geometry>
         <mesh filename="package://otim_traj/model/cam_support/CAM_support.STL" scale="0.001 0.001 0.001"/>
@@ -50,9 +50,9 @@
     <parent link="wrist_2_link"/>
     <child link="CAM_support_link"/>
-  </joint>
+  </joint> -->
   ########################################
   # Realsense code
   ########################################
-  <sensor_d435 parent="CAM_support_link">
+  <!-- <sensor_d435 parent="CAM_support_link">
     <origin xyz="-0.0277 -0.002 -0.0075" rpy="0 0 0"/>
   </sensor_d435>
@@ -62,5 +62,5 @@
     <child link="d435_realsense"/>
     <origin xyz="0.0 0.0 0.0" rpy="0.0 0.0 0.0"/>
-  </joint>
+  </joint> -->
   ########################################
   # Robotiq code

Commit message: add moveit config working with stomp and chomp & add gitignore file

File: otim_traj/urdf/ur5_grasp.urdf.xacro (robot description, xacro)
@@ -15,5 +15,5 @@
   <xacro:ur5_robot prefix="" joint_limited="false" transmission_hw_interface="$(arg transmission_hw_interface)"/>
   <link name="world"/>
-  <joint name="world_joint" type="fixed">
+  <joint name="world" type="fixed">
     <parent link="world"/>
     <child link="base_link"/>
